Commit message: Adding vrx 2.2 changes

File: vrx_urdf/wamv_gazebo/urdf/components/wamv_gps.xacro (robot description, xacro)
@@ -2,5 +2,5 @@
 <robot xmlns:xacro="http://ros.org/wiki/xacro">
   <xacro:macro name="wamv_gps" params="name:=gps x:=0.3 y:=0 z:=1.3
-				       R:=0 P:=0 Y:=0 update_rate:=15">
+				       R:=0 P:=0 Y:=0 update_rate:=20">
     <link name="${namespace}/${name}_link">
       <visual name="${name}_visual">
@@ -37,5 +37,5 @@
       <sensor name="navsat" type="navsat">
         <always_on>1</always_on>
-        <update_rate>15</update_rate>
+        <update_rate>20</update_rate>
         <!--<topic>${namespace}/${sensor_namespace}gps/gps/fix</topic>-->
       </sensor>

File: vrx_urdf/wamv_gazebo/urdf/components/wamv_imu.xacro (robot description, xacro)
@@ -1,5 +1,5 @@
 <?xml version="1.0"?>
 <robot xmlns:xacro="http://ros.org/wiki/xacro">
-  <xacro:macro name="wamv_imu" params="name:=imu x:=0.3 y:=0.5 z:=1.3 R:=0 P:=0 Y:=0 update_rate:=15">
+  <xacro:macro name="wamv_imu" params="name:=imu x:=0.3 y:=0.5 z:=1.3 R:=0 P:=0 Y:=0 update_rate:=20">
     <link name="${namespace}/${name}_link">
       <visual name="${name}_visual">>

File: vrx_urdf/wamv_gazebo/urdf/thruster_layouts/wamv_gazebo_thruster_config.xacro (robot description, xacro)
@@ -14,5 +14,5 @@
       <propeller_diameter>0.2</propeller_diameter>
       <velocity_control>true</velocity_control>
-      <!-- max total thrust / 2 -->
+      <!-- max total thrust / 2 = 305-->
       <max_thrust_cmd>${((x_u + x_uu * max_velocity_mps) * max_velocity_mps)/ 2}</max_thrust_cmd>
       <namespace>${namespace}</namespace>
